Commit message: dave with eyes, goggles, imu in proper position

File: simws/src/gpg3_gazebo/urdf/gopi5go_dave.urdf (robot description, URDF)
Before this commit: robot gopi5go_dave, 7 links, 6 joints
Links:
- added link dave_eyes_link; visual cylinder length=0.001 radius=0.005; visual cylinder length=0.001 radius=0.005
- link gopi5go_dave_link: geometry visual cylinder length=0.008 radius=0.015; visual cylinder length=0.008 radius=0.015
Joints:
- added joint joint_dave_eyes: type fixed, parent base_link, child dave_eyes_link, origin xyz=-0.04 0 0.250 rpy=0 0 0
- joint joint_imu: origin xyz=0.070 0.035 0.055 rpy=0 0 0 -> xyz=0.070 0.035 0.104 rpy=0 0 0
