Commit message: temp use waffle as model GoPiGo3

File: simws/src/gpg3_gazebo/urdf/gpg3_gopigo3.urdf (robot description, URDF)
Before this commit: robot gpg3_gopigo3, 7 links, 6 joints
Links:
- removed link caster_back_link
- added link camera_depth_frame
- added link camera_depth_optical_frame
- added link camera_link; collision box size=0.012 0.132 0.020; visual mesh filename=package://gpg3_gazebo/models/gpg3_common/meshes/r200.dae
- added link camera_rgb_frame
- added link camera_rgb_optical_frame
- added link caster_back_left_link, mass 0.005; collision box size=0.030 0.009 0.020
- added link caster_back_right_link, mass 0.005; collision box size=0.030 0.009 0.020
- link base_link: mass 8.2573504e-01 -> 1.3729096e+00; geometry collision box size=0.266 0.266 0.094; visual mesh filename=package://gpg3_gazebo/models/gpg3_common/meshes/gopigo3_bas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 scale=0.001 0.001 0.001
Joints:
- removed joint caster_back_joint
- added joint camera_depth_joint: type fixed, parent camera_link, child camera_depth_frame, origin xyz=0.005 0.028 0.013 rpy=0 0 0
- added joint camera_depth_optical_joint: type fixed, parent camera_depth_frame, child camera_depth_optical_frame, origin xyz=0 0 0 rpy=-1.57 0 -1.57
- added joint camera_joint: type fixed, parent base_link, child camera_link, origin xyz=0.064 -0.065 0.094 rpy=0 0 0
- added joint camera_rgb_joint: type fixed, parent camera_link, child camera_rgb_frame, origin xyz=0.005 0.018 0.013 rpy=0 0 0
- added joint camera_rgb_optical_joint: type fixed, parent camera_rgb_frame, child camera_rgb_optical_frame, origin xyz=0 0 0 rpy=-1.57 0 -1.57
- added joint caster_back_left_joint: type fixed, parent base_link, child caster_back_left_link, origin xyz=-0.177 0.064 -0.004 rpy=-1.57 0 0
- added joint caster_back_right_joint: type fixed, parent base_link, child caster_back_right_link, origin xyz=-0.177 -0.064 -0.004 rpy=-1.57 0 0
- joint base_joint: origin xyz=0.0 0.0 0.010 rpy=0 0 0 -> xyz=0 0 0.010 rpy=0 0 0
- joint imu_joint: origin xyz=-0.032 0 0.068 rpy=0 0 0 -> xyz=0.0 0 0.068 rpy=0 0 0
- joint scan_joint: origin xyz=-0.032 0 0.172 rpy=0 0 0 -> xyz=-0.064 0 0.122 rpy=0 0 0
- joint wheel_left_joint: origin xyz=0.0 0.08 0.023 rpy=-1.57 0 0 -> xyz=0.0 0.144 0.023 rpy=-1.57 0 0
- joint wheel_right_joint: origin xyz=0.0 -0.080 0.023 rpy=-1.57 0 0 -> xyz=0.0 -0.144 0.023 rpy=-1.57 0 0
