Commit message: collision with z to lift it off floor, now responds to cmd_vel topics correctly

File: simws/src/gpg3_gazebo/urdf/gpg3_gopi5go_dave.urdf (robot description, URDF)
Before this commit: robot gopi5go_dave, 8 links, 7 joints
Links:
- removed link laser_frame
- removed link left_wheel
- removed link right_wheel
- added link base_footprint
- added link base_scan; visual cylinder length=0.020 radius=0.0325
- added link wheel_left_link, mass 0.1; collision cylinder length=0.025 radius=0.03385; visual cylinder length=0.025 radius=0.03385
- added link wheel_right_link; visual cylinder length=0.025 radius=0.033385
- link base_link: mass None -> 1.13; geometry collision box size=0.23 0.14 0.37; visual box size=0.025 0.055 0.002
Joints:
- removed joint joint_left_wheel
- removed joint joint_right_wheel
- added joint base_joint: type fixed, parent base_footprint, child base_link, origin xyz=0 0 0 rpy=0 0 0
- added joint wheel_left_joint: type continuous, parent base_link, child wheel_left_link, origin xyz=0 0.058 0.033385 rpy=-1.57 0 0, axis 0 0 1
- added joint wheel_right_joint: type continuous, parent base_link, child wheel_right_link, origin xyz=0 -0.058 0.033385 rpy=-1.57 0 0, axis 0 0 1
- joint joint_ydlidar: child laser_frame -> base_scan

Commit message: seems to be working

File: simws/src/gpg3_gazebo/urdf/gpg3_gopi5go_dave.urdf (robot description, URDF)
Before this commit: robot gopi5go_dave, 9 links, 8 joints
Links:
- added link rear_castor_link; visual sphere radius=0.01
- link base_link: geometry collision box size=0.23 0.14 0.37; visual box size=0.025 0.055 0.002
Joints:
- added joint rear_castor_joint: type fixed, parent base_link, child rear_castor_link, origin xyz=-0.114 0 0.01 rpy=0 0 0

Commit message: caster joint set to fixed for simplicity to keep ball moving with bot

File: simws/src/gpg3_gazebo/urdf/gpg3_gopi5go_dave.urdf (robot description, URDF)
Before this commit: robot gopi5go_dave, 10 links, 9 joints
Links:
- removed link rear_castor_link
- added link rear_caster_link; visual sphere radius=0.01
Joints:
- removed joint rear_castor_joint
- added joint rear_caster_joint: type fixed, parent base_link, child rear_caster_link, origin xyz=-0.114 0 0.01 rpy=0 0 0

Commit message: sim looks good but rviz model wheels and castor problems

File: simws/src/gpg3_gazebo/urdf/gpg3_gopi5go_dave.urdf (robot description, URDF)
Before this commit: robot gopi5go_dave, 10 links, 9 joints
Links:
- removed link oak_d_w_frame
- added link camera_link; collision box size=0.022 0.097 0.030; visual box size=0.022 0.097 0.030
- added link camera_rgb_frame
Joints:
- removed joint joint_oak_d_w
- added joint camera_joint: type fixed, parent base_link, child camera_link, origin xyz=0.08 0 0.162 rpy=0 0 0
- added joint camera_rgb_joint: type fixed, parent camera_link, child camera_rgb_frame

Commit message: cleaned up wayward caster wheel

File: simws/src/gpg3_gazebo/urdf/gpg3_gopi5go_dave.urdf (robot description, URDF)
Before this commit: robot gopi5go_dave, 11 links, 10 joints
Links:
- removed link rear_caster_link
- link base_link: geometry collision box size=0.23 0.14 0.37; visual box size=0.025 0.055 0.002
Joints:
- removed joint rear_caster_joint
- joint wheel_left_joint: axis 0 0 1 -> 0 1 0; origin xyz=0 0.058 0.033385 rpy=-1.57 0 0 -> xyz=0 0.058 0.033385 rpy=0 0 0
- joint wheel_right_joint: axis 0 0 1 -> 0 1 0; origin xyz=0 -0.058 0.033385 rpy=-1.57 0 0 -> xyz=0 -0.058 0.033385 rpy=0 0 0
